File: PT4115_CWW_Driver.kicad_pcb (KiCad board)
At the start: 2 copper layers, 20 x 24 mm, 31 parts, among them P1 LED, P2 DIM, P3 PWR, U1 PT4115, U2 PT4115

Commit message: Gerber Output
Parts:
- added REF**: Via_0406, BK_Common:Via_0406, F.Cu at (68.6, 67.4)
- added REF**: Via_0406, BK_Common:Via_0406, F.Cu at (66.6, 61.2)
- added REF**: Via_0406, BK_Common:Via_0406, F.Cu at (59.3, 68.2)
- added REF**: Via_0406, BK_Common:Via_0406, F.Cu at (60.0, 61.9)
- added REF**: Via_0406, BK_Common:Via_0406, F.Cu at (56.6, 61.1)
- moved C1 70.7 mm to (52.1, 52.0)
- moved C2 70.7 mm to (67.3, 52.0)
- moved C3 70.7 mm to (63.4, 60.6)
- moved C4 70.7 mm to (53.5, 60.6)
- moved C5 70.7 mm to (51.1, 64.8)
- moved C6 70.7 mm to (61.1, 64.9)
- moved D1 70.7 mm to (58.3, 57.3)
- moved D2 70.7 mm to (68.1, 57.3)
- moved L1 70.7 mm to (53.4, 56.7)
- moved L2 70.7 mm to (63.2, 56.7)
- moved P1 70.7 mm to (55.9, 52.0)
- moved P2 70.7 mm to (52.1, 71.9)
- moved P3 70.7 mm to (67.6, 71.9)
- moved R1 70.7 mm to (58.8, 63.7)
- moved R2 70.7 mm to (68.9, 63.8)
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Routing:
- net /Out2P: track 25.6 -> 29.5 mm
- net /Out1N: track 13.4 -> 11.1 mm
- net /VIN: track 54.0 -> 55.6 mm
- net Net-(D2-Pad2): track 10.6 -> 12.1 mm
- net Net-(D1-Pad2): track 10.6 -> 11.8 mm
- net /Out1P: track 26.1 -> 26.7 mm
Other:
- board text added: "PT4115 2Ch LED Driver v1.0 BK 2017"
- board text added: "PT4115_2Ch V1.0 BK2017"
- board text removed: "PT4115 2Ch LED Driver v1.0 BK 20017"
- board text removed: "PT4115_2Ch BK2017"
